Commit message: [urdf] Added a DoF to shoulders + head

File: urdf/human-tpl.xacro (robot description, xacro)
@@ -5,4 +5,6 @@
     <xacro:property name="neck_shoulder_length" value="0.3" />
     <xacro:property name="torso_height" value="0.8" />
+    <xacro:property name="head_radius" value="0.2" />
+    <xacro:property name="neck_length" value="0.1" />
     <xacro:property name="arm_radius" value="0.025" />
     <link name="neck">
@@ -14,5 +16,38 @@
         </visual>
     </link>
-    <xacro:macro name="arm_segment" params="name reflect length parent attachment_origin attachment_rotation link_name">
+    <link name="head_r">
+    </link>
+    <link name="head_p">
+    </link>
+    <link name="head">
+        <visual>
+            <geometry>
+                <sphere radius="${head_radius}"/>
+            </geometry>
+            <origin rpy="0 0 0" xyz="0 0 ${head_radius}" />
+        </visual>
+    </link>
+    <joint name="head_r" type="revolute">
+        <axis xyz="1 0 0" />
+        <limit effort="1000" lower="-1." upper="1." velocity="0.5" />
+        <parent link="neck"/>
+        <child link="head_r"/>
+        <origin rpy="0 0 0" xyz="0 0 ${neck_length}" />
+    </joint>
+    <joint name="head_p" type="revolute">
+        <axis xyz="0 -1 0" />
+        <limit effort="1000" lower="-1.4" upper="1.4" velocity="0.5" />
+        <parent link="head_r"/>
+        <child link="head_p"/>
+        <origin rpy="0 0 0" xyz="0 0 0" />
+    </joint>
+    <joint name="head_y" type="revolute">
+        <axis xyz="0 0 1" />
+        <limit effort="1000" lower="-1.5" upper="1.5" velocity="0.5" />
+        <parent link="head_p"/>
+        <child link="head"/>
+        <origin rpy="0 0 0" xyz="0 0 0" />
+    </joint>
+    <xacro:macro name="arm_segment" params="name reflect length parent attachment_origin attachment_rotation link_name link_min_limit link_max_limit">
         <link name="${name}">
             <visual>
@@ -24,6 +59,6 @@
         </link>
         <joint name="${link_name}" type="revolute">
-            <axis xyz="0 1 0" />
-            <limit effort="1000" lower="-1.7" upper="1.5" velocity="0.5" />
+            <axis xyz="0 -1 0" />
+            <limit effort="1000" lower="${link_min_limit}" upper="${link_max_limit}" velocity="0.5" />
             <parent link="${parent}"/>
             <child link="${name}"/>
@@ -32,11 +67,22 @@
     </xacro:macro>
     <xacro:macro name="arm" params="suffix parent reflect">
+        <link name="${suffix}_z_shoulder">
+        </link>
+        <joint name="${suffix}_z_shoulder" type="revolute">
+            <axis xyz="0 0 ${reflect * -1}" />
+            <limit effort="1000" lower="-1.8" upper="2.5" velocity="0.5" />
+            <parent link="${parent}"/>
+            <child link="${suffix}_z_shoulder"/>
+            <origin rpy="0 0 ${reflect * 1.57}" xyz="0 ${reflect * neck_shoulder_length} 0" />
+        </joint>
         <xacro:arm_segment name="${suffix}_upperarm"
                      length = "${upperarm_length}"
                      reflect="${reflect}"
-                     parent="${parent}"
-                     attachment_origin="0 ${reflect * neck_shoulder_length} 0"
-                     attachment_rotation="0 0 ${reflect * 1.57}"
-                     link_name="${suffix}_shoulder" />
+                     parent="${suffix}_z_shoulder"
+                     attachment_origin="0 0 0"
+                     attachment_rotation="0 0 0"
+                     link_name="${suffix}_y_shoulder"
+                     link_min_limit="-1.5"
+                     link_max_limit="1.7" />
         <xacro:arm_segment name="${suffix}_forearm"
                      length = "${forearm_length}"
@@ -45,5 +91,7 @@
                      attachment_origin="${upperarm_length} 0 0"
                      attachment_rotation="0 0 0"
-                     link_name="${suffix}_elbow" />
+                     link_name="${suffix}_elbow"
+                     link_min_limit="0"
+                     link_max_limit="2.5" />
     </xacro:macro>
     <xacro:arm suffix="l" reflect="1" parent="neck" />

Commit message: Added a body_ frame + body ID suffixes everywhere
This follows the ROS4HRI convention

File: urdf/human-tpl.xacro (robot description, xacro)
@@ -1,4 +1,5 @@
 <?xml version="1.0"?>
 <robot xmlns:xacro="http://www.ros.org/wiki/xacro" name="human">
+    <xacro:property name="id" value="03d4" />
     <xacro:property name="upperarm_length" value="0.4" />
     <xacro:property name="forearm_length" value="0.45" />
@@ -8,5 +9,7 @@
     <xacro:property name="neck_length" value="0.1" />
     <xacro:property name="arm_radius" value="0.025" />
-    <link name="neck">
+    <link name="body_${id}">
+    </link>
+    <link name="torso_${id}">
         <visual>
             <geometry>
@@ -16,9 +19,15 @@
         </visual>
     </link>
-    <link name="head_r">
+    <joint name="torso_${id}" type="fixed">
+        <axis xyz="0 0 1" />
+        <parent link="body_${id}"/>
+        <child link="torso_${id}"/>
+        <origin rpy="0 0 0" xyz="0 0 ${torso_height}" />
+    </joint>
+    <link name="head_r_${id}">
     </link>
-    <link name="head_p">
+    <link name="head_p_${id}">
     </link>
-    <link name="head">
+    <link name="head_${id}">
         <visual>
             <geometry>
@@ -28,23 +37,23 @@
         </visual>
     </link>
-    <joint name="head_r" type="revolute">
+    <joint name="head_r_${id}" type="revolute">
         <axis xyz="1 0 0" />
         <limit effort="1000" lower="-1." upper="1." velocity="0.5" />
-        <parent link="neck"/>
-        <child link="head_r"/>
+        <parent link="torso_${id}"/>
+        <child link="head_r_${id}"/>
         <origin rpy="0 0 0" xyz="0 0 ${neck_length}" />
     </joint>
-    <joint name="head_p" type="revolute">
+    <joint name="head_p_${id}" type="revolute">
         <axis xyz="0 -1 0" />
         <limit effort="1000" lower="-1.4" upper="1.4" velocity="0.5" />
-        <parent link="head_r"/>
-        <child link="head_p"/>
+        <parent link="head_r_${id}"/>
+        <child link="head_p_${id}"/>
         <origin rpy="0 0 0" xyz="0 0 0" />
     </joint>
-    <joint name="head_y" type="revolute">
+    <joint name="head_y_${id}" type="revolute">
         <axis xyz="0 0 1" />
         <limit effort="1000" lower="-1.5" upper="1.5" velocity="0.5" />
-        <parent link="head_p"/>
-        <child link="head"/>
+        <parent link="head_p_${id}"/>
+        <child link="head_${id}"/>
         <origin rpy="0 0 0" xyz="0 0 0" />
     </joint>
@@ -67,11 +76,11 @@
     </xacro:macro>
     <xacro:macro name="arm" params="suffix parent reflect">
-        <link name="${suffix}_z_shoulder">
+        <link name="${suffix}_y_shoulder_${id}">
         </link>
-        <joint name="${suffix}_z_shoulder" type="revolute">
+        <joint name="${suffix}_z_shoulder_${id}" type="revolute">
             <axis xyz="0 0 ${reflect * -1}" />
             <limit effort="1000" lower="-1.8" upper="2.5" velocity="0.5" />
             <parent link="${parent}"/>
-            <child link="${suffix}_z_shoulder"/>
+            <child link="${suffix}_y_shoulder_${id}"/>
             <origin rpy="0 0 ${reflect * 1.57}" xyz="0 ${reflect * neck_shoulder_length} 0" />
         </joint>
@@ -79,8 +88,8 @@
                      length = "${upperarm_length}"
                      reflect="${reflect}"
-                     parent="${suffix}_z_shoulder"
+                     parent="${suffix}_y_shoulder_${id}"
                      attachment_origin="0 0 0"
                      attachment_rotation="0 0 0"
-                     link_name="${suffix}_y_shoulder"
+                     link_name="${suffix}_p_shoulder_${id}"
                      link_min_limit="-1.5"
                      link_max_limit="1.7" />
@@ -91,9 +100,9 @@
                      attachment_origin="${upperarm_length} 0 0"
                      attachment_rotation="0 0 0"
-                     link_name="${suffix}_elbow"
+                     link_name="${suffix}_elbow_${id}"
                      link_min_limit="0"
                      link_max_limit="2.5" />
     </xacro:macro>
-    <xacro:arm suffix="l" reflect="1" parent="neck" />
-    <xacro:arm suffix="r" reflect="-1" parent="neck" />
+    <xacro:arm suffix="l" reflect="1" parent="torso_${id}" />
+    <xacro:arm suffix="r" reflect="-1" parent="torso_${id}" />
 </robot>

Commit message: [urdf] Added a simple script showing how to generate the URDF from Python

File: urdf/human-tpl.xacro (robot description, xacro)
@@ -1,7 +1,7 @@
 <?xml version="1.0"?>
 <robot xmlns:xacro="http://www.ros.org/wiki/xacro" name="human">
-    <xacro:property name="id" value="03d4" />
-    <xacro:property name="upperarm_length" value="0.4" />
-    <xacro:property name="forearm_length" value="0.45" />
+    <xacro:property name="id" value="$(arg id)" />
+    <xacro:property name="upperarm_length" value="$(arg upperarm_length)" />
+    <xacro:property name="forearm_length" value="$(arg forearm_length)" />
     <xacro:property name="neck_shoulder_length" value="0.3" />
     <xacro:property name="torso_height" value="0.8" />
@@ -83,5 +83,5 @@
             <parent link="${parent}"/>
             <child link="${suffix}_y_shoulder_${id}"/>
-            <origin rpy="0 0 ${reflect * 1.57}" xyz="0 ${reflect * neck_shoulder_length} 0" />
+            <origin rpy="0 0 ${reflect * pi / 2}" xyz="0 ${reflect * neck_shoulder_length} 0" />
         </joint>
         <xacro:arm_segment name="${suffix}_upperarm"

Commit message: Added the legs

File: urdf/human-tpl.xacro (robot description, xacro)
@@ -1,12 +1,38 @@
 <?xml version="1.0"?>
 <robot xmlns:xacro="http://www.ros.org/wiki/xacro" name="human">
+    <!-- User-settable parameters (eg, xacro human-tpl.xacro id:=xyz) -->
     <xacro:property name="id" value="$(arg id)" />
+    <xacro:property name="head_radius" value="$(arg head_radius)" />
+    <xacro:property name="neck_length" value="$(arg neck_length)" />
+    <xacro:property name="neck_shoulder_length" value="$(arg neck_shoulder_length)" />
     <xacro:property name="upperarm_length" value="$(arg upperarm_length)" />
     <xacro:property name="forearm_length" value="$(arg forearm_length)" />
-    <xacro:property name="neck_shoulder_length" value="0.3" />
-    <xacro:property name="torso_height" value="0.8" />
-    <xacro:property name="head_radius" value="0.2" />
-    <xacro:property name="neck_length" value="0.1" />
-    <xacro:property name="arm_radius" value="0.025" />
+    <xacro:property name="torso_height" value="$(arg torso_height)" />
+    <xacro:property name="waist_length" value="$(arg waist_length)" />
+    <xacro:property name="tight_length" value="$(arg tight_length)" />
+    <xacro:property name="tibia_length" value="$(arg tibia_length)" />
+    <!-- Parameters defaults -->
+    <xacro:arg name="id" default="default" />
+    <xacro:arg name="head_radius" default="0.15" />
+    <xacro:arg name="neck_length" default="0.1" />
+    <xacro:arg name="neck_shoulder_length" default="0.2" />
+    <xacro:arg name="upperarm_length" default="0.2" />
+    <xacro:arg name="forearm_length" default="0.3" />
+    <xacro:arg name="torso_height" default="0.5" />
+    <xacro:arg name="waist_length" default="0.3" />
+    <xacro:arg name="tight_length" default="0.4" />
+    <xacro:arg name="tibia_length" default="0.4" />
+    <xacro:property name="arm_radius" value="0.04" />
+    <!-- Materials -->
+    <material name="yellow-skin">
+        <color rgba="1 0.7 0 1" />
+    </material>
+    <material name="yellow-skin-dark">
+        <color rgba="0.9 0.6 0 1" />
+    </material>
+    <material name="black">
+        <color rgba="0 0 0 1" />
+    </material>
+    <!--***********-->
     <link name="body_${id}">
     </link>
@@ -14,6 +40,14 @@
         <visual>
             <geometry>
-                <box size="0.2 ${neck_shoulder_length * 2} ${torso_height}"/>
-            </geometry>
+                <box size="0.25 ${neck_shoulder_length * 2} ${torso_height/3}"/>
+            </geometry>
+            <material name="yellow-skin" />
+            <origin rpy="0 0 0" xyz="0 0 ${-torso_height/6 + arm_radius}" />
+        </visual>
+        <visual>
+            <geometry>
+                <box size="0.2 ${neck_shoulder_length * 1.5} ${torso_height}"/>
+            </geometry>
+            <material name="yellow-skin" />
             <origin rpy="0 0 0" xyz="0 0 -${torso_height/2}" />
         </visual>
@@ -27,5 +61,5 @@
     <link name="head_r_${id}">
     </link>
-    <link name="head_p_${id}">
+    <link name="head_y_${id}">
     </link>
     <link name="head_${id}">
@@ -34,5 +68,21 @@
                 <sphere radius="${head_radius}"/>
             </geometry>
+            <material name="yellow-skin" />
             <origin rpy="0 0 0" xyz="0 0 ${head_radius}" />
+        </visual>
+        <!-- eyes -->
+        <visual>
+            <geometry>
+                <sphere radius="${head_radius/5}"/>
+            </geometry>
+            <material name="black" />
+            <origin rpy="0 0 0" xyz="${head_radius * .9} ${2*head_radius/5} ${head_radius}" />
+        </visual>
+        <visual>
+            <geometry>
+                <sphere radius="${head_radius/5}"/>
+            </geometry>
+            <material name="black" />
+            <origin rpy="0 0 0" xyz="${head_radius * .9} -${2*head_radius/5} ${head_radius}" />
         </visual>
     </link>
@@ -44,29 +94,37 @@
         <origin rpy="0 0 0" xyz="0 0 ${neck_length}" />
     </joint>
+    <joint name="head_y_${id}" type="revolute">
+        <axis xyz="0 0 1" />
+        <limit effort="1000" lower="-1.4" upper="1.4" velocity="0.5" />
+        <parent link="head_r_${id}"/>
+        <child link="head_y_${id}"/>
+        <origin rpy="0 0 0" xyz="0 0 0" />
+    </joint>
     <joint name="head_p_${id}" type="revolute">
         <axis xyz="0 -1 0" />
-        <limit effort="1000" lower="-1.4" upper="1.4" velocity="0.5" />
-        <parent link="head_r_${id}"/>
-        <child link="head_p_${id}"/>
-        <origin rpy="0 0 0" xyz="0 0 0" />
-    </joint>
-    <joint name="head_y_${id}" type="revolute">
-        <axis xyz="0 0 1" />
         <limit effort="1000" lower="-1.5" upper="1.5" velocity="0.5" />
-        <parent link="head_p_${id}"/>
+        <parent link="head_y_${id}"/>
         <child link="head_${id}"/>
         <origin rpy="0 0 0" xyz="0 0 0" />
     </joint>
-    <xacro:macro name="arm_segment" params="name reflect length parent attachment_origin attachment_rotation link_name link_min_limit link_max_limit">
+    <xacro:macro name="limb_segment" params="name reflect length parent attachment_origin attachment_rotation link_name link_axis link_min_limit link_max_limit">
         <link name="${name}">
             <visual>
                 <geometry>
-                    <box size="${length} ${arm_radius * 2} ${arm_radius * 2}"/>
+                    <cylinder length="${length}" radius="${arm_radius}"/>
                 </geometry>
-                <origin rpy="0 0 0" xyz="${length/2} 0 0" />
+                <material name="yellow-skin" />
+                <origin rpy="0 ${pi/2} 0" xyz="${length/2} 0 0" />
+            </visual>
+            <visual>
+                <geometry>
+                    <sphere radius="${1.5 * arm_radius}"/>
+                </geometry>
+                <material name="yellow-skin" />
+                <origin rpy="0 0 0" xyz="${length} 0 0" />
             </visual>
         </link>
         <joint name="${link_name}" type="revolute">
-            <axis xyz="0 -1 0" />
+            <axis xyz="${link_axis}" />
             <limit effort="1000" lower="${link_min_limit}" upper="${link_max_limit}" velocity="0.5" />
             <parent link="${parent}"/>
@@ -77,6 +135,13 @@
     <xacro:macro name="arm" params="suffix parent reflect">
         <link name="${suffix}_y_shoulder_${id}">
+            <visual>
+            <geometry>
+                <sphere radius="${2 * arm_radius}"/>
+            </geometry>
+            <material name="yellow-skin-dark" />
+            <origin rpy="0 0 0" xyz="0 0 0" />
+        </visual>
         </link>
-        <joint name="${suffix}_z_shoulder_${id}" type="revolute">
+        <joint name="${suffix}_y_shoulder_${id}" type="revolute">
             <axis xyz="0 0 ${reflect * -1}" />
             <limit effort="1000" lower="-1.8" upper="2.5" velocity="0.5" />
@@ -85,5 +150,5 @@
             <origin rpy="0 0 ${reflect * pi / 2}" xyz="0 ${reflect * neck_shoulder_length} 0" />
         </joint>
-        <xacro:arm_segment name="${suffix}_upperarm"
+        <xacro:limb_segment name="${suffix}_upperarm_${id}"
                      length = "${upperarm_length}"
                      reflect="${reflect}"
@@ -92,13 +157,15 @@
                      attachment_rotation="0 0 0"
                      link_name="${suffix}_p_shoulder_${id}"
-                     link_min_limit="-1.5"
+                     link_axis="0 -1 0"
+                     link_min_limit="-2.5"
                      link_max_limit="1.7" />
-        <xacro:arm_segment name="${suffix}_forearm"
+         <xacro:limb_segment name="${suffix}_forearm_${id}"
                      length = "${forearm_length}"
                      reflect="${reflect}"
-                     parent="${suffix}_upperarm"
+                     parent="${suffix}_upperarm_${id}"
                      attachment_origin="${upperarm_length} 0 0"
                      attachment_rotation="0 0 0"
                      link_name="${suffix}_elbow_${id}"
+                     link_axis="0 -1 0"
                      link_min_limit="0"
                      link_max_limit="2.5" />
@@ -106,3 +173,43 @@
     <xacro:arm suffix="l" reflect="1" parent="torso_${id}" />
     <xacro:arm suffix="r" reflect="-1" parent="torso_${id}" />
+    <xacro:macro name="leg" params="suffix parent reflect">
+        <link name="${suffix}_r_hip_${id}">
+            <visual>
+            <geometry>
+                <sphere radius="${2 * arm_radius}"/>
+            </geometry>
+            <material name="yellow-skin-dark" />
+            <origin rpy="0 0 0" xyz="0 0 0" />
+        </visual>
+        </link>
+        <joint name="${suffix}_r_hip_${id}" type="revolute">
+            <axis xyz="0 ${reflect * -1} 0" />
+            <limit effort="1000" lower="-.2" upper="1." velocity="0.5" />
+            <parent link="${parent}"/>
+            <child link="${suffix}_r_hip_${id}"/>
+            <origin rpy="${reflect * pi/2} ${pi/2} ${pi}" xyz="0 ${reflect * waist_length/2} -${torso_height}" />
+        </joint>
+        <xacro:limb_segment name="${suffix}_tight_${id}"
+                     length = "${tight_length}"
+                     reflect="${reflect}"
+                     parent="${suffix}_r_hip_${id}"
+                     attachment_origin="0 0 0"
+                     attachment_rotation="0 0 0"
+                     link_name="${suffix}_p_hip_${id}"
+                     link_axis="0 0 ${-reflect}"
+                     link_min_limit="-.5"
+                     link_max_limit="1.8" />
+        <xacro:limb_segment name="${suffix}_tibia_${id}"
+                     length = "${tibia_length}"
+                     reflect="${reflect}"
+                     parent="${suffix}_tight_${id}"
+                     attachment_origin="${tight_length} 0 0"
+                     attachment_rotation="0 0 0"
+                     link_name="${suffix}_knee_${id}"
+                     link_axis="0 0 ${-reflect}"
+                     link_min_limit="-2.5"
+                     link_max_limit="0" />
+    </xacro:macro>
+    <xacro:leg suffix="l" reflect="1" parent="torso_${id}" />
+    <xacro:leg suffix="r" reflect="-1" parent="torso_${id}" />
 </robot>

Commit message: [urdf] Added 1 DoF at waist + fix orientation r hip

File: urdf/human-tpl.xacro (robot description, xacro)
@@ -37,4 +37,6 @@
     <link name="body_${id}">
     </link>
+    <link name="waist_${id}">
+    </link>
     <link name="torso_${id}">
         <visual>
@@ -54,8 +56,14 @@
     </link>
     <joint name="torso_${id}" type="fixed">
-        <axis xyz="0 0 1" />
-        <parent link="body_${id}"/>
+        <parent link="waist_${id}"/>
         <child link="torso_${id}"/>
         <origin rpy="0 0 0" xyz="0 0 ${torso_height}" />
+    </joint>
+    <joint name="waist_${id}" type="revolute">
+        <axis xyz="0 1 0" />
+        <limit effort="1000" lower="-.2" upper="1." velocity="0.5" />
+        <parent link="body_${id}"/>
+        <child link="waist_${id}"/>
+        <origin rpy="0 0 0" xyz="0 0 0" />
     </joint>
     <link name="head_r_${id}">
@@ -184,9 +192,9 @@
         </link>
         <joint name="${suffix}_r_hip_${id}" type="revolute">
-            <axis xyz="0 ${reflect * -1} 0" />
+            <axis xyz="0 -1 0" />
             <limit effort="1000" lower="-.2" upper="1." velocity="0.5" />
             <parent link="${parent}"/>
             <child link="${suffix}_r_hip_${id}"/>
-            <origin rpy="${reflect * pi/2} ${pi/2} ${pi}" xyz="0 ${reflect * waist_length/2} -${torso_height}" />
+            <origin rpy="${reflect * pi/2} ${pi/2} ${pi}" xyz="0 ${reflect * waist_length/2} 0" />
         </joint>
         <xacro:limb_segment name="${suffix}_tight_${id}"
@@ -211,5 +219,5 @@
                      link_max_limit="0" />
     </xacro:macro>
-    <xacro:leg suffix="l" reflect="1" parent="torso_${id}" />
-    <xacro:leg suffix="r" reflect="-1" parent="torso_${id}" />
+    <xacro:leg suffix="l" reflect="1" parent="body_${id}" />
+    <xacro:leg suffix="r" reflect="-1" parent="body_${id}" />
 </robot>
