Commit message: [urdf] added hand + foot links + shoulder roll

File: urdf/human-tpl.xacro (robot description, xacro)
@@ -158,14 +158,23 @@
             <origin rpy="0 0 ${reflect * pi / 2}" xyz="0 ${reflect * neck_shoulder_length} 0" />
         </joint>
+        <link name="${suffix}_p_shoulder_${id}">
+        </link>
+        <joint name="${suffix}_p_shoulder_${id}" type="revolute">
+            <axis xyz="0 -1 0" />
+            <limit effort="1000" lower="-2.5" upper="1.7" velocity="0.5" />
+            <parent link="${suffix}_y_shoulder_${id}"/>
+            <child link="${suffix}_p_shoulder_${id}"/>
+            <origin rpy="0 0 0" xyz="0 0 0" />
+        </joint>
         <xacro:limb_segment name="${suffix}_upperarm_${id}"
                      length = "${upperarm_length}"
                      reflect="${reflect}"
-                     parent="${suffix}_y_shoulder_${id}"
+                     parent="${suffix}_p_shoulder_${id}"
                      attachment_origin="0 0 0"
                      attachment_rotation="0 0 0"
-                     link_name="${suffix}_p_shoulder_${id}"
-                     link_axis="0 -1 0"
-                     link_min_limit="-2.5"
-                     link_max_limit="1.7" />
+                     link_name="${suffix}_r_shoulder_${id}"
+                     link_axis="${reflect} 0 0"
+                     link_min_limit="-1.7"
+                     link_max_limit="1.5" />
          <xacro:limb_segment name="${suffix}_forearm_${id}"
                      length = "${forearm_length}"
@@ -175,7 +184,14 @@
                      attachment_rotation="0 0 0"
                      link_name="${suffix}_elbow_${id}"
-                     link_axis="0 -1 0"
+                     link_axis="0 0 ${-reflect}"
                      link_min_limit="0"
                      link_max_limit="2.5" />
+        <link name="${suffix}_hand_${id}">
+        </link>
+        <joint name="${suffix}_wrist_${id}" type="fixed">
+            <parent link="${suffix}_forearm_${id}"/>
+            <child link="${suffix}_hand_${id}"/>
+            <origin rpy="0 0 0" xyz="${forearm_length} 0 0" />
+        </joint>
     </xacro:macro>
     <xacro:arm suffix="l" reflect="1" parent="torso_${id}" />
@@ -218,4 +234,11 @@
                      link_min_limit="-2.5"
                      link_max_limit="0" />
+        <link name="${suffix}_foot_${id}">
+        </link>
+        <joint name="${suffix}_ankle_${id}" type="fixed">
+            <parent link="${suffix}_tibia_${id}"/>
+            <child link="${suffix}_foot_${id}"/>
+            <origin rpy="0 0 0" xyz="${tibia_length} 0 0" />
+        </joint>
     </xacro:macro>
     <xacro:leg suffix="l" reflect="1" parent="body_${id}" />

Commit message: [urdf] Adjust range of shoulder pitch

File: urdf/human-tpl.xacro (robot description, xacro)
@@ -162,5 +162,5 @@
         <joint name="${suffix}_p_shoulder_${id}" type="revolute">
             <axis xyz="0 -1 0" />
-            <limit effort="1000" lower="-2.5" upper="1.7" velocity="0.5" />
+            <limit effort="1000" lower="-1.3" upper="1.7" velocity="0.5" />
             <parent link="${suffix}_y_shoulder_${id}"/>
             <child link="${suffix}_p_shoulder_${id}"/>

Commit message: WIP on xacro model

File: urdf/human-tpl.xacro (robot description, xacro)
@@ -3,24 +3,19 @@
     <!-- User-settable parameters (eg, xacro human-tpl.xacro id:=xyz) -->
     <xacro:property name="id" value="$(arg id)" />
-    <xacro:property name="head_radius" value="$(arg head_radius)" />
-    <xacro:property name="neck_length" value="$(arg neck_length)" />
-    <xacro:property name="neck_shoulder_length" value="$(arg neck_shoulder_length)" />
-    <xacro:property name="upperarm_length" value="$(arg upperarm_length)" />
-    <xacro:property name="forearm_length" value="$(arg forearm_length)" />
-    <xacro:property name="torso_height" value="$(arg torso_height)" />
-    <xacro:property name="waist_length" value="$(arg waist_length)" />
-    <xacro:property name="tight_length" value="$(arg tight_length)" />
-    <xacro:property name="tibia_length" value="$(arg tibia_length)" />
+    <xacro:property name="height" value="$(arg height)" />
     <!-- Parameters defaults -->
     <xacro:arg name="id" default="default" />
-    <xacro:arg name="head_radius" default="0.15" />
-    <xacro:arg name="neck_length" default="0.1" />
-    <xacro:arg name="neck_shoulder_length" default="0.2" />
-    <xacro:arg name="upperarm_length" default="0.2" />
-    <xacro:arg name="forearm_length" default="0.3" />
-    <xacro:arg name="torso_height" default="0.5" />
-    <xacro:arg name="waist_length" default="0.3" />
-    <xacro:arg name="tight_length" default="0.4" />
-    <xacro:arg name="tibia_length" default="0.4" />
+    <xacro:arg name="height" default="1.65" />
+    <!-- human body proportions taken from https://www.thedrawingsource.com/figure-drawing-proportions.html -->
+    <xacro:property name="size_unit" value="${height/7.5}" />
+    <xacro:property name="head_radius" value="${size_unit/2}" />
+    <xacro:property name="neck_length" value="${size_unit * 0.25}" />
+    <xacro:property name="neck_shoulder_length" value="${size_unit*0.8}" />
+    <xacro:property name="upperarm_length" value="${size_unit*1.6}" />
+    <xacro:property name="forearm_length" value="${size_unit}" />
+    <xacro:property name="torso_height" value="${size_unit*2.75}" />
+    <xacro:property name="waist_length" value="${size_unit*1.2}" />
+    <xacro:property name="tight_length" value="${size_unit*1.5}" />
+    <xacro:property name="tibia_length" value="${size_unit*2}" />
     <xacro:property name="arm_radius" value="0.04" />
     <!-- Materials -->
@@ -214,5 +209,5 @@
             <origin rpy="${reflect * pi/2} ${pi/2} ${pi}" xyz="0 ${reflect * waist_length/2} 0" />
         </joint>
-        <xacro:limb_segment name="${suffix}_tight_${id}"
+        <xacro:limb_segment name="${suffix}_hip_${id}"
                      length = "${tight_length}"
                      reflect="${reflect}"
@@ -224,5 +219,5 @@
                      link_min_limit="-.5"
                      link_max_limit="1.8" />
-        <xacro:limb_segment name="${suffix}_tibia_${id}"
+        <xacro:limb_segment name="${suffix}_knee_${id}"
                      length = "${tibia_length}"
                      reflect="${reflect}"

Commit message: Updated xacro model to comply with REP 103 and 120

File: urdf/human-tpl.xacro (robot description, xacro)
@@ -37,16 +37,25 @@
         <visual>
             <geometry>
-                <box size="0.25 ${neck_shoulder_length * 2} ${torso_height/3}"/>
-            </geometry>
-            <material name="yellow-skin" />
-            <origin rpy="0 0 0" xyz="0 0 ${-torso_height/6 + arm_radius}" />
-        </visual>
-        <visual>
-            <geometry>
-                <box size="0.2 ${neck_shoulder_length * 1.5} ${torso_height}"/>
+                <sphere radius="${waist_length/2}"/>
+            </geometry>
+            <material name="yellow-skin" />
+            <origin rpy="0 0 0" xyz="0 0 -${torso_height*2/3}" />
+        </visual>
+        <visual>
+            <geometry>
+                <sphere radius="${neck_shoulder_length}"/>
+            </geometry>
+            <material name="yellow-skin" />
+            <origin rpy="0 0 0" xyz="0 0 -${torso_height/4}" />
+        </visual>
+        <!--
+        <visual>
+            <geometry>
+                <box size="0.2 ${waist_length * 1.2} ${torso_height}"/>
             </geometry>
             <material name="yellow-skin" />
             <origin rpy="0 0 0" xyz="0 0 -${torso_height/2}" />
         </visual>
+        -->
     </link>
     <joint name="torso_${id}" type="fixed">
@@ -66,4 +75,6 @@
     <link name="head_y_${id}">
     </link>
+    <link name="head_p_${id}">
+    </link>
     <link name="head_${id}">
         <visual>
@@ -72,5 +83,5 @@
             </geometry>
             <material name="yellow-skin" />
-            <origin rpy="0 0 0" xyz="0 0 ${head_radius}" />
+            <origin rpy="0 0 0" xyz="${-head_radius/2} 0 0" />
         </visual>
         <!-- eyes -->
@@ -80,5 +91,5 @@
             </geometry>
             <material name="black" />
-            <origin rpy="0 0 0" xyz="${head_radius * .9} ${2*head_radius/5} ${head_radius}" />
+            <origin rpy="0 0 0" xyz="${head_radius * .9 - head_radius/2} ${2*head_radius/5} 0" />
         </visual>
         <visual>
@@ -87,5 +98,5 @@
             </geometry>
             <material name="black" />
-            <origin rpy="0 0 0" xyz="${head_radius * .9} -${2*head_radius/5} ${head_radius}" />
+            <origin rpy="0 0 0" xyz="${head_radius * .9 - head_radius/2} -${2*head_radius/5} 0" />
         </visual>
     </link>
@@ -108,6 +119,11 @@
         <limit effort="1000" lower="-1.5" upper="1.5" velocity="0.5" />
         <parent link="head_y_${id}"/>
+        <child link="head_p_${id}"/>
+        <origin rpy="0 0 0" xyz="0 0 0" />
+    </joint>
+    <joint name="head_${id}" type="fixed">
+        <parent link="head_p_${id}"/>
         <child link="head_${id}"/>
-        <origin rpy="0 0 0" xyz="0 0 0" />
+        <origin rpy="0 0 0" xyz="${head_radius/2} 0 ${head_radius}" />
     </joint>
     <xacro:macro name="limb_segment" params="name reflect length parent attachment_origin attachment_rotation link_name link_axis link_min_limit link_max_limit">
@@ -118,5 +134,5 @@
                 </geometry>
                 <material name="yellow-skin" />
-                <origin rpy="0 ${pi/2} 0" xyz="${length/2} 0 0" />
+                <origin rpy="0 0 0" xyz="0 0 -${length/2}" />
             </visual>
             <visual>
@@ -125,5 +141,5 @@
                 </geometry>
                 <material name="yellow-skin" />
-                <origin rpy="0 0 0" xyz="${length} 0 0" />
+                <origin rpy="0 0 0" xyz="0 0 -${length}" />
             </visual>
         </link>
@@ -148,14 +164,14 @@
         <joint name="${suffix}_y_shoulder_${id}" type="revolute">
             <axis xyz="0 0 ${reflect * -1}" />
-            <limit effort="1000" lower="-1.8" upper="2.5" velocity="0.5" />
+            <limit effort="1000" lower="-1.7" upper="1.1" velocity="0.5" />
             <parent link="${parent}"/>
             <child link="${suffix}_y_shoulder_${id}"/>
-            <origin rpy="0 0 ${reflect * pi / 2}" xyz="0 ${reflect * neck_shoulder_length} 0" />
+            <origin rpy="0 0 0" xyz="0 ${reflect * neck_shoulder_length} 0" />
         </joint>
         <link name="${suffix}_p_shoulder_${id}">
         </link>
         <joint name="${suffix}_p_shoulder_${id}" type="revolute">
-            <axis xyz="0 -1 0" />
-            <limit effort="1000" lower="-1.3" upper="1.7" velocity="0.5" />
+            <axis xyz="${reflect} 0 0" />
+            <limit effort="1000" lower="-0.4" upper="3.3" velocity="0.5" />
             <parent link="${suffix}_y_shoulder_${id}"/>
             <child link="${suffix}_p_shoulder_${id}"/>
@@ -169,5 +185,5 @@
                      attachment_rotation="0 0 0"
                      link_name="${suffix}_r_shoulder_${id}"
-                     link_axis="${reflect} 0 0"
+                     link_axis="0 0 ${reflect}"
                      link_min_limit="-1.7"
                      link_max_limit="1.5" />
@@ -176,16 +192,16 @@
                      reflect="${reflect}"
                      parent="${suffix}_upperarm_${id}"
-                     attachment_origin="${upperarm_length} 0 0"
+                     attachment_origin="0 0 -${upperarm_length}"
                      attachment_rotation="0 0 0"
                      link_name="${suffix}_elbow_${id}"
-                     link_axis="0 0 ${-reflect}"
+                     link_axis="0 -1 0"
                      link_min_limit="0"
                      link_max_limit="2.5" />
-        <link name="${suffix}_hand_${id}">
+        <link name="${suffix}_wrist_${id}">
         </link>
         <joint name="${suffix}_wrist_${id}" type="fixed">
             <parent link="${suffix}_forearm_${id}"/>
-            <child link="${suffix}_hand_${id}"/>
-            <origin rpy="0 0 0" xyz="${forearm_length} 0 0" />
+            <child link="${suffix}_wrist_${id}"/>
+            <origin rpy="0 0 0" xyz="0 0 -${forearm_length}" />
         </joint>
     </xacro:macro>
@@ -193,5 +209,5 @@
     <xacro:arm suffix="r" reflect="-1" parent="torso_${id}" />
     <xacro:macro name="leg" params="suffix parent reflect">
-        <link name="${suffix}_r_hip_${id}">
+        <link name="${suffix}_y_hip_${id}">
             <visual>
             <geometry>
@@ -202,37 +218,37 @@
         </visual>
         </link>
-        <joint name="${suffix}_r_hip_${id}" type="revolute">
-            <axis xyz="0 -1 0" />
-            <limit effort="1000" lower="-.2" upper="1." velocity="0.5" />
+        <joint name="${suffix}_y_hip_${id}" type="revolute">
+            <axis xyz="0 0 -1" />
+            <limit effort="1000" lower="-.1" upper="0.6" velocity="0.5" />
             <parent link="${parent}"/>
-            <child link="${suffix}_r_hip_${id}"/>
-            <origin rpy="${reflect * pi/2} ${pi/2} ${pi}" xyz="0 ${reflect * waist_length/2} 0" />
+            <child link="${suffix}_y_hip_${id}"/>
+            <origin rpy="0 0 0" xyz="0 ${reflect * waist_length/2} 0" />
         </joint>
         <xacro:limb_segment name="${suffix}_hip_${id}"
                      length = "${tight_length}"
                      reflect="${reflect}"
-                     parent="${suffix}_r_hip_${id}"
+                     parent="${suffix}_y_hip_${id}"
                      attachment_origin="0 0 0"
                      attachment_rotation="0 0 0"
                      link_name="${suffix}_p_hip_${id}"
-                     link_axis="0 0 ${-reflect}"
-                     link_min_limit="-.5"
-                     link_max_limit="1.8" />
+                     link_axis="0 -1 0"
+                     link_min_limit="-.4"
+                     link_max_limit="0.7" />
         <xacro:limb_segment name="${suffix}_knee_${id}"
                      length = "${tibia_length}"
                      reflect="${reflect}"
-                     parent="${suffix}_tight_${id}"
-                     attachment_origin="${tight_length} 0 0"
+                     parent="${suffix}_hip_${id}"
+                     attachment_origin="0 0 -${tight_length}"
                      attachment_rotation="0 0 0"
                      link_name="${suffix}_knee_${id}"
-                     link_axis="0 0 ${-reflect}"
+                     link_axis="0 -1 0"
                      link_min_limit="-2.5"
                      link_max_limit="0" />
-        <link name="${suffix}_foot_${id}">
+        <link name="${suffix}_ankle_${id}">
         </link>
         <joint name="${suffix}_ankle_${id}" type="fixed">
-            <parent link="${suffix}_tibia_${id}"/>
-            <child link="${suffix}_foot_${id}"/>
-            <origin rpy="0 0 0" xyz="${tibia_length} 0 0" />
+            <parent link="${suffix}_knee_${id}"/>
+            <child link="${suffix}_ankle_${id}"/>
+            <origin rpy="0 0 0" xyz="0 0 -${tibia_length}" />
         </joint>
     </xacro:macro>

Commit message: [urdf] upperarm->shoulder, forearm->elbow

File: urdf/human-tpl.xacro (robot description, xacro)
@@ -178,5 +178,5 @@
             <origin rpy="0 0 0" xyz="0 0 0" />
         </joint>
-        <xacro:limb_segment name="${suffix}_upperarm_${id}"
+        <xacro:limb_segment name="${suffix}_shoulder_${id}"
                      length = "${upperarm_length}"
                      reflect="${reflect}"
@@ -188,8 +188,8 @@
                      link_min_limit="-1.7"
                      link_max_limit="1.5" />
-         <xacro:limb_segment name="${suffix}_forearm_${id}"
+         <xacro:limb_segment name="${suffix}_elbow_${id}"
                      length = "${forearm_length}"
                      reflect="${reflect}"
-                     parent="${suffix}_upperarm_${id}"
+                     parent="${suffix}_shoulder_${id}"
                      attachment_origin="0 0 -${upperarm_length}"
                      attachment_rotation="0 0 0"
@@ -201,5 +201,5 @@
         </link>
         <joint name="${suffix}_wrist_${id}" type="fixed">
-            <parent link="${suffix}_forearm_${id}"/>
+            <parent link="${suffix}_elbow_${id}"/>
             <child link="${suffix}_wrist_${id}"/>
             <origin rpy="0 0 0" xyz="0 0 -${forearm_length}" />
